File: esp32-tft+gps.sch (EAGLE design)
At the start: 36 parts, among them IC1 TCAN1051HGV, J4 Vertical Qwiic Connector, U2 XN04312, U8 NCP1117LPST50T3G

Commit message: actually save
Parts:
- removed -_+_G_V_T_R_E_0, -_+_G_V_T_R_E_1: MF-CON-2.54mm-01x08, SparkFun-Connectors:M081X08
- removed C_SER, POW12, POW5: (no value), MF_Passives:CAPACITOR_NP_0603
- removed D2: BAS16, SparkFun-DiscreteSemi:DIODEBAS16
- removed IC1: TCAN1051HGV, microbuilder:CAN_TRANSCIEVER_TCAN1051V
- removed JP1: DB9, SparkFun-Connectors:DB9FEMALE
- removed R1, R3, RCAN: (no value), 00jim:RESISTOR_0603
- removed U2: XN04312, SparkFun-DiscreteSemi:XN04312SOT
- removed U3: (no value), SparkFun-IC-Power:V_REG_78XXSINK
- added J5: (no value), SparkFun-Connectors:CONN_02
Connections:
- removed net CAN_H: IC1.CANH, JP1.1, RCAN.P$2
- removed net CAN_L: IC1.CANL, JP1.2, RCAN.P$1
- removed net N$4: C_SER.P$1, D2.A, R3.P$1
- removed net RAW: -_+_G_V_T_R_E_0.2, -_+_G_V_T_R_E_1.2, JP1.7, JP1.8, POW12.P$1, U3.IN
- removed net RS-IN: D2.C, JP1.5, U2.B1
- removed net RS-OUT: JP1.4, R3.P$2, U2.C2
- removed net UNITID: -_+_G_V_T_R_E_0.4, -_+_G_V_T_R_E_1.4, JP1.3
- net CANRX: no longer IC1.RXD
- net CANTX: no longer IC1.TXD
- net CAN_S: no longer IC1.S
- net DB9_RX: no longer U2.B2
- net DB9_TX: no longer R1.P$1, U2.C1
- net GND: no longer C_SER.P$2, IC1.GND, U2.E1
- net GND_HC: now also J5.1; no longer -_+_G_V_T_R_E_0.1, -_+_G_V_T_R_E_1.1, JP1.6, JP1.9, POW12.P$2, POW5.P$2, U3.GND
- net RX2: no longer -_+_G_V_T_R_E_0.7, -_+_G_V_T_R_E_1.8
- net RX3: no longer -_+_G_V_T_R_E_0.5, -_+_G_V_T_R_E_1.6
- net TX2: no longer -_+_G_V_T_R_E_0.8, -_+_G_V_T_R_E_1.7
- net TX3: no longer -_+_G_V_T_R_E_0.6, -_+_G_V_T_R_E_1.5
- net VCC: no longer IC1.VIO, R1.P$2, U2.E2
- net VCC_50: now also J5.2; no longer -_+_G_V_T_R_E_0.3, -_+_G_V_T_R_E_1.3, IC1.+5V, POW5.P$1, U3.OUT

Commit message: Add touchscreen header directly to board
Parts:
- added U$4: SPI_TFT_TOUCH, 00jim:SPI_TFT_TOUCH
Connections:
- removed net CANRX: U$3.GPIO16
- removed net CANTX: U$3.GPIO15
- removed net CAN_S: U$3.GPIO17
- removed net CLK: J3.5
- removed net DB9_RX: U$3.GPIO26
- removed net DB9_TX: U$3.GPIO27
- removed net RX0: J1.4
- removed net RX2: U$3.GPIO39
- removed net RX3: U$3.GPIO34
- removed net TX0: J1.3
- removed net TX2: U$3.GPIO25
- removed net TX3: U$3.GPIO13
- net GND: now also U$4.GND
- net LED: now also U$3.GPIO13
- net MISO: now also U$4.S_MISO, U$4.T_DO
- net MOSI: now also U$4.S_MOSI, U$4.T_DIN
- net RXI: now also J1.4
- net SCLK: now also J3.5, U$4.S_SCK, U$4.T_CLK
- net TCH_CS: now also U$4.T_CS
- net TFT_CS: now also U$4.S_CS
- net TFT_DC: now also U$4.S_DC
- net TXO: now also J1.3
- net VCC: now also U$4.LED, U$4.S_RESET, U$4.VCC
