File: integrated_winglevlr_pow_and_cpu.sch (EAGLE design)
At the start: 13 parts

Commit message: Add I2C connector
Parts:
- added I2C: Vertical Qwiic Connector, SparkFun-Connectors:QWIIC_CONNECTOR
Connections:
- net GND: now also I2C.1
- net SCL1: now also I2C.4
- net SDA1: now also I2C.3
- net VCC_33: now also I2C.2
Changed lines of the file:
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@@
 <part name="CAP2" library="SparkFun-Connectors" deviceset="CONN_02" device=""/>
 <part name="BAT1" library="SparkFun-Connectors" deviceset="CONN_02" device=""/>
+<part name="I2C" library="SparkFun-Connectors" deviceset="QWIIC_CONNECTOR" device="" value="Vertical Qwiic Connector"/>
 </parts>
 <sheets>
@@
 <attribute name="NAME" x="10.16" y="-22.352" size="1.778" layer="95" font="vector"/>
 </instance>
+<instance part="I2C" gate="G$1" x="-30.48" y="-20.32" smashed="yes">
+<attribute name="NAME" x="-35.56" y="-12.446" size="1.778" layer="95" font="vector"/>
+</instance>
 </instances>
 <busses>
@@
 <label x="20.32" y="-27.94" size="1.778" layer="95"/>
 </segment>
+<segment>
+<wire x1="-22.86" y1="-22.86" x2="-15.24" y2="-22.86" width="0.1524" layer="91"/>
+<label x="-20.32" y="-22.86" size="1.778" layer="95"/>
+<pinref part="I2C" gate="G$1" pin="1"/>
+</segment>
 </net>
 <net name="VCHARGE" class="0">
@@
 <label x="-12.7" y="40.64" size="1.778" layer="95"/>
 </segment>
+<segment>
+<wire x1="-22.86" y1="-20.32" x2="-15.24" y2="-20.32" width="0.1524" layer="91"/>
+<label x="-20.32" y="-20.32" size="1.778" layer="95"/>
+<pinref part="I2C" gate="G$1" pin="2"/>
+</segment>
 </net>
 <net name="GPS_TX" class="0">
@@
 <label x="-48.26" y="20.32" size="1.778" layer="95"/>
 </segment>
+<segment>
+<wire x1="-22.86" y1="-15.24" x2="-15.24" y2="-15.24" width="0.1524" layer="91"/>
+<label x="-20.32" y="-15.24" size="1.778" layer="95"/>
+<pinref part="I2C" gate="G$1" pin="4"/>
+</segment>
 </net>
 <net name="SDA1" class="0">
@@
 <label x="-48.26" y="25.4" size="1.778" layer="95"/>
 </segment>
-</net>
+<segment>
+<wire x1="-22.86" y1="-17.78" x2="-15.24" y2="-17.78" width="0.1524" layer="91"/>
+<label x="-20.32" y="-17.78" size="1.778" layer="95"/>
+<pinref part="I2C" gate="G$1" pin="3"/>
+</segment>
+</net>
