File: servo_power.brd (EAGLE design)
At the start: 34 x 31.7 mm, 17 parts, among them T1 2N3904

Commit message: PEC11D rotary encoder test chip
Parts:
- removed R2: (no value), 00jim:R1206
- removed R3, R5, R7: 100k, 00jim:R1206
- removed R4, R6: 10k, 00jim:R1206
- removed SV2: (no value), con-lstb:MA06-1
- added -+12EPP: (no value), con-lstb:MA08-1
- added B1D, B2D: 10k, 00jim:R1206
- added B1U, B2U, FETU, G1: 100k, 00jim:R1206
- added SV3: (no value), con-lstb:MA03-1
- moved SV1 1.27 mm to (30.5, 26.7)
Connections:
- removed net PWM: SV1.3, SV2.6
- new net NC1: -+12EPP.8
- new net PWM1: -+12EPP.6, SV1.3
- new net PWM2: -+12EPP.7, SV3.3
- net GND: now also -+12EPP.1, B1D.P$2, B2D.P$2, SV3.1; no longer R4.P$2, R6.P$2, SV2.1
- net N$13: now also G1.P$2; no longer R2.P$2
- net N$15: now also FETU.P$2; no longer R7.P$2
- net SRVEN: now also -+12EPP.5, G1.P$1; no longer R2.P$1, SV2.5
- net VBAT1: now also B1U.P$1; no longer R3.P$1
- net VBAT2: now also B2U.P$1; no longer R5.P$1
- net VCC50: now also -+12EPP.2; no longer SV2.2
- net VSENS1: now also -+12EPP.3, B1D.P$1, B1U.P$2; no longer R3.P$2, R4.P$1, SV2.3
- net VSENS2: now also -+12EPP.4, B2D.P$1, B2U.P$2; no longer R5.P$2, R6.P$1, SV2.4
- net VSERV: now also FETU.P$1; no longer R7.P$1
- net VSERVS: now also SV3.2
Routing:
- net GND: track 0.00 -> 89.9 mm
- net VBAT2: track 0.00 -> 43.7 mm
- net VCC50: track 0.00 -> 34.7 mm
- net VSERV: track 0.00 -> 30.5 mm
- net VBAT1: track 0.00 -> 24.0 mm
- net VBATS: track 0.00 -> 20.7 mm
- net VSERVS: track 0.00 -> 20.1 mm
- net SRVEN: track 0.00 -> 17.1 mm
- net N$15: track 0.00 -> 16.7 mm
- net PWM1: track 0.00 -> 15.5 mm
- net VSENS1: track 0.00 -> 13.6 mm
- net PWM2: track 0.00 -> 13.0 mm
- net VCHG: track 0.00 -> 13.0 mm
- net VSENS2: track 0.00 -> 9.36 mm
- net N$13: track 0.00 -> 3.84 mm
